File: circuit/機電整合.kicad_pcb (KiCad board)
At the start: 2 copper layers, 105 x 64.9 mm, 37 parts, among them J1 Screw_Terminal_01x02, J10 Conn_01x03, J11 Conn_01x03, J12 Conn_01x03, J13 Conn_01x03, J14 Conn_01x06, J15 Screw_Terminal_01x02, J16 Screw_Terminal_01x02, J17 Screw_Terminal_01x02, J18 Screw_Terminal_01x02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

Commit message: k
Parts:
- U3, U4, U5, U6, U7: footprint Package_DIP:DIP-16_W7.62mm -> Package_DIP:DIP-16_W7.62mm_Socket
