File: circuit/機電整合.kicad_pcb (KiCad board)
At the start: 2 copper layers, 7 parts, among them U1 L293D, U2 74HC595, U3 74HC595, U4 L293D, U5 L293D, U6 ESP32-CAM

Commit message: nano pinout
Parts:
- added D1: LED, LED_THT:LED_D3.0mm_FlatTop, F.Cu at (135.6, 48.7)
- added D2: LED, LED_THT:LED_D3.0mm_FlatTop, F.Cu at (135.6, 54.3)
- added D3: LED, LED_THT:LED_D3.0mm_FlatTop, F.Cu at (135.6, 59.8)
- added J1: Conn_01x08, Connector_PinHeader_2.54mm:PinHeader_1x08_P2.54mm_Vertical, F.Cu at (142.2, 48.3)
- added R1: 200, LED_THT:LED_D3.0mm_FlatTop, F.Cu at (135.6, 65.4)
- added R2: 200, LED_THT:LED_D3.0mm_FlatTop, F.Cu at (135.6, 70.9)
- added R3: 200, LED_THT:LED_D3.0mm_FlatTop, F.Cu at (135.6, 76.5)
Connections:
- net /motorLb- renamed /motorLB-
- A1 pad 1: unconnected-(A1-D1/TX-Pad1) -> Net-(A1-D1/TX)
- A1 pad 12: unconnected-(A1-D9-Pad12) -> /nano_D9
- A1 pad 15: unconnected-(A1-D12-Pad15) -> /nano_D12
- A1 pad 16: unconnected-(A1-D13-Pad16) -> /nano_D13
- A1 pad 19: unconnected-(A1-A0-Pad19) -> /nano_A0
- A1 pad 2: unconnected-(A1-D0/RX-Pad2) -> /nano_RX
- A1 pad 20: unconnected-(A1-A1-Pad20) -> /nano_A1
- A1 pad 21: unconnected-(A1-A2-Pad21) -> /nano_A2
- A1 pad 22: unconnected-(A1-A3-Pad22) -> /nano_A3
- A1 pad 25: unconnected-(A1-A6-Pad25) -> /nano_A6
- A1 pad 26: unconnected-(A1-A7-Pad26) -> /nano_A7
- A1 pad 3: unconnected-(A1-~{RESET}-Pad3) -> /nano_reset
- A1 pad 5: unconnected-(A1-D2-Pad5) -> /nano_D2
- A1 pad 8: unconnected-(A1-D5-Pad8) -> /nano_D5
- A1 pad 9: unconnected-(A1-D6-Pad9) -> /nano_D6
- U1 pad 8: +12V -> +5V
- U4 pad 8: +12V -> +5V
- U5 pad 8: +12V -> +5V
- U6 pad 11: unconnected-(U6-IO0-Pad11) -> /esp32_GPI0
- U6 pad 12: unconnected-(U6-GND_2-Pad12) -> GND
- U6 pad 14: unconnected-(U6-U0R-Pad14) -> /esp32_RX
- U6 pad 15: unconnected-(U6-U0T-Pad15) -> /esp32_TX
- U6 pad 7: unconnected-(U6-GND_1-Pad7) -> GND

Commit message: update
Parts:
- added C1: C, Capacitor_THT:C_Disc_D5.0mm_W2.5mm_P5.00mm, F.Cu at (61.5, 60.1)
- added C2: C, Capacitor_THT:C_Disc_D5.0mm_W2.5mm_P5.00mm, F.Cu at (77.5, 59.6)
- added C3: C, Capacitor_THT:C_Disc_D5.0mm_W2.5mm_P5.00mm, F.Cu at (127.2, 60.9)
- added J10: Conn_01x03, Connector_PinHeader_2.54mm:PinHeader_1x03_P2.54mm_Vertical, F.Cu at (123.3, 120.9)
- added J11: Conn_01x03, Connector_PinHeader_2.54mm:PinHeader_1x03_P2.54mm_Vertical, F.Cu at (128.0, 120.9)
- added J12: Conn_01x03, Connector_PinHeader_2.54mm:PinHeader_1x03_P2.54mm_Vertical, F.Cu at (132.6, 120.9)
- added J13: Conn_01x03, Connector_PinHeader_2.54mm:PinHeader_1x03_P2.54mm_Vertical, F.Cu at (137.3, 120.9)
- added J14: Conn_01x06, Connector_PinHeader_2.54mm:PinHeader_1x06_P2.54mm_Vertical, F.Cu at (91.4, 78.7)
- added J15: Screw_Terminal_01x02, Connector:HANDSON_KF301-2P, F.Cu at (38.1, 58.4)
- added J16: Conn_01x08, Connector_PinHeader_2.54mm:PinHeader_1x08_P2.54mm_Vertical, F.Cu at (132.1, 73.7)
- added J17: Conn_01x08, Connector_PinHeader_2.54mm:PinHeader_1x08_P2.54mm_Vertical, F.Cu at (137.2, 73.7)
- added J2: Screw_Terminal_01x02, Connector:HANDSON_KF301-2P, F.Cu at (71.2, 37.2)
- added J3: Screw_Terminal_01x02, Connector:HANDSON_KF301-2P, F.Cu at (94.0, 37.2)
- added J4: Screw_Terminal_01x02, Connector:HANDSON_KF301-2P, F.Cu at (38.1, 45.7)
- added J5: Screw_Terminal_01x02, Connector:HANDSON_KF301-2P, F.Cu at (53.6, 37.3)
- added J6: Screw_Terminal_01x02, Connector:HANDSON_KF301-2P, F.Cu at (112.8, 37.6)
- added J7: Screw_Terminal_01x02, Connector:HANDSON_KF301-2P, F.Cu at (136.7, 61.0)
- added J8: Conn_01x03, Connector_PinHeader_2.54mm:PinHeader_1x03_P2.54mm_Vertical, F.Cu at (114.0, 120.9)
- added J9: Conn_01x03, Connector_PinHeader_2.54mm:PinHeader_1x03_P2.54mm_Vertical, F.Cu at (118.7, 120.9)
- added R4: 1k, Resistor_THT:R_Axial_DIN0309_L9.0mm_D3.2mm_P12.70mm_Horizontal, F.Cu at (94.0, 127.1)
- added U7: LM7805_TO220, Package_TO_SOT_THT:TO-220-3_Vertical, F.Cu at (35.6, 71.1)
- R1, R2, R3: footprint LED_THT:LED_D3.0mm_FlatTop -> Resistor_THT:R_Axial_DIN0207_L6.3mm_D2.5mm_P7.62mm_Horizontal
- moved U6 156.9 mm to (12.7, -2.54)
- moved R3 69.1 mm to (81.9, 120.0)
- moved U4 57.4 mm to (50.8, 53.5)
- moved D1 52.5 mm to (157.5, 96.4)
- moved D2 52.5 mm to (157.5, 102.0)
- moved D3 52.5 mm to (157.5, 107.5)
- moved J1 52.3 mm to (101.6, 81.3), turned to 90 degrees
- moved A1 41.8 mm to (79.5, 77.2), turned to -90 degrees
- moved U5 27.1 mm to (116.8, 53.3)
- moved U3 21.3 mm to (108.8, 71.1), turned to 180 degrees
- moved R1 21.2 mm to (154.7, 74.6)
- moved R2 20.0 mm to (151.3, 83.5)
- moved U1 16.6 mm to (67.1, 53.3), turned to 0 degrees
- moved U2 7.37 mm to (83.6, 53.3)
Connections:
- A1 pad 17: +3.3V -> unconnected-(A1-3V3-Pad17)
- A1 pad 30: +12V -> unconnected-(A1-VIN-Pad30)
- U6 pad 11: /esp32_GPI0 -> unconnected-(U6-IO0-Pad11)
- U6 pad 12: GND -> unconnected-(U6-GND_2-Pad12)
- U6 pad 14: /esp32_RX -> unconnected-(U6-U0R-Pad14)
- U6 pad 15: /esp32_TX -> unconnected-(U6-U0T-Pad15)
- U6 pad 16: GND -> unconnected-(U6-GND_3-Pad16)
- U6 pad 4: /SDA -> unconnected-(U6-IO15-Pad4)
- U6 pad 5: /SCL -> unconnected-(U6-IO13-Pad5)
- U6 pad 7: GND -> unconnected-(U6-GND_1-Pad7)
- U6 pad 8: +5V -> unconnected-(U6-5V-Pad8)
- U6 pad 9: +3.3V -> unconnected-(U6-3V3-Pad9)
Other:
- board outline added: 108.2 x 63.1 mm

Commit message: pcb done
Parts:
- removed the J1 at (101.6, 81.3)
- removed U1: L293D, Package_DIP:DIP-16_W7.62mm
- removed the U2 at (83.6, 53.3)
- added J4: Conn_01x02, Connector_PinHeader_2.54mm:PinHeader_1x02_P2.54mm_Vertical, F.Cu at (111.8, 74.9)
- added J5: Conn_01x02, Connector_PinHeader_2.54mm:PinHeader_1x02_P2.54mm_Vertical, F.Cu at (111.1, 71.1)
- added J6: Conn_01x02, Connector_PinHeader_2.54mm:PinHeader_1x02_P2.54mm_Vertical, F.Cu at (82.5, 69.8)
- added J7: Conn_01x02, Connector_PinHeader_2.54mm:PinHeader_1x02_P2.54mm_Vertical, F.Cu at (123.2, 74.9)
- added U3: 74HC595, Package_DIP:DIP-16_W7.62mm, F.Cu at (68.6, 48.3)
- C1: value C -> 10uf; footprint Capacitor_THT:C_Disc_D5.0mm_W2.5mm_P5.00mm -> Capacitor_THT:CP_Radial_D5.0mm_P2.50mm
- C2: renamed from C3; value C -> 10uf; footprint Capacitor_THT:C_Disc_D5.0mm_W2.5mm_P5.00mm -> Capacitor_THT:CP_Radial_D5.0mm_P2.50mm
- C3: renamed from C2; value C -> 10uf; footprint Capacitor_THT:C_Disc_D5.0mm_W2.5mm_P5.00mm -> Capacitor_THT:CP_Radial_D5.0mm_P2.50mm
- R1: renamed from R4; footprint Resistor_THT:R_Axial_DIN0309_L9.0mm_D3.2mm_P12.70mm_Horizontal -> Resistor_THT:R_Axial_DIN0207_L6.3mm_D2.5mm_P10.16mm_Horizontal
- R2: renamed from R1; value 200 -> 220; footprint Resistor_THT:R_Axial_DIN0207_L6.3mm_D2.5mm_P7.62mm_Horizontal -> Resistor_THT:R_Axial_DIN0207_L6.3mm_D2.5mm_P10.16mm_Horizontal
- R3: renamed from R2; value 200 -> 220; footprint Resistor_THT:R_Axial_DIN0207_L6.3mm_D2.5mm_P7.62mm_Horizontal -> Resistor_THT:R_Axial_DIN0207_L6.3mm_D2.5mm_P10.16mm_Horizontal
- R4: renamed from R3; value 200 -> 220; footprint Resistor_THT:R_Axial_DIN0207_L6.3mm_D2.5mm_P7.62mm_Horizontal -> Resistor_THT:R_Axial_DIN0207_L6.3mm_D2.5mm_P10.16mm_Horizontal
- U6: value ESP32-CAM -> L293D; footprint Module:ESP32-CAM -> Package_DIP:DIP-16_W7.62mm
- moved D1 115.4 mm to (42.5, 87.0), turned to -90 degrees
- moved R2 112.5 mm to (42.5, 84.5), turned to 90 degrees
- moved U6 87.4 mm to (83.8, 48.3)
- moved D2 72.0 mm to (121.9, 39.4), turned to 180 degrees
- moved R4 68.2 mm to (129.5, 71.1), turned to 180 degrees
- moved R1 57.7 mm to (101.6, 69.8), turned to 180 degrees
- moved R3 50.1 mm to (120.7, 43.8)
- moved J8 49.1 mm to (100.3, 73.7), turned to 90 degrees
- moved D3 49.0 mm to (129.5, 67.3), turned to 90 degrees
- moved J9 47.1 mm to (100.3, 77.5), turned to 90 degrees
- moved J13 46.5 mm to (100.3, 92.7), turned to 90 degrees
- moved J10 45.8 mm to (100.3, 81.3), turned to 90 degrees
- moved J12 45.4 mm to (100.3, 88.9), turned to 90 degrees
- moved J11 45.2 mm to (100.3, 85.1), turned to 90 degrees
- moved J14 31.3 mm to (63.5, 92.7), turned to 90 degrees
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- renumbered J15 to J1, J2 to J15, J3 to J16, J4 to J17, J5 to J18, J6 to J19, J16 to J2, J7 to J20, J17 to J3, U7 to U2, U3 to U4, U4 to U5, U5 to U7
Connections:
- C1 pad 1: GND -> +12V
- C1 pad 2: +12V -> GND
- C2 pad 1: GND -> +12V
- C2 pad 2: +12V -> GND
- C3 pad 1: GND -> +12V
- C3 pad 2: +12V -> GND
- U6 pad 1: unconnected-(U6-IO4-Pad1) -> /wheel_speed
- U6 pad 10: unconnected-(U6-IO16-Pad10) -> /motor2_A
- U6 pad 11: unconnected-(U6-IO0-Pad11) -> /motorRF+
- U6 pad 12: unconnected-(U6-GND_2-Pad12) -> GND
- U6 pad 13: unconnected-(U6-VCC-Pad13) -> GND
- U6 pad 14: unconnected-(U6-U0R-Pad14) -> /motorRF-
- U6 pad 15: unconnected-(U6-U0T-Pad15) -> /motor2_B
- U6 pad 16: unconnected-(U6-GND_3-Pad16) -> +12V
- U6 pad 2: unconnected-(U6-IO2-Pad2) -> /motor1_A
- U6 pad 3: unconnected-(U6-IO14-Pad3) -> /motorLF+
- U6 pad 4: unconnected-(U6-IO15-Pad4) -> GND
- U6 pad 5: unconnected-(U6-IO13-Pad5) -> GND
- U6 pad 6: unconnected-(U6-IO12-Pad6) -> /motorLF-
- U6 pad 7: unconnected-(U6-GND_1-Pad7) -> /motor1_B
- U6 pad 8: unconnected-(U6-5V-Pad8) -> +5V
- U6 pad 9: unconnected-(U6-3V3-Pad9) -> /wheel_speed
Routing:
- net GND: track 0.00 -> 363.0 mm
- net +5V: track 0.00 -> 268.2 mm
- net /wheel_speed: track 0.00 -> 147.2 mm
- net /motor6_speed: track 0.00 -> 122.5 mm
- net +12V: track 0.00 -> 118.4 mm
- net /motor5_speed: track 0.00 -> 84.3 mm
- net /motor2_A: track 0.00 -> 59.3 mm
- net /SDA: track 0.00 -> 58.5 mm
- net /SCL: track 0.00 -> 58.5 mm
- net /nano_D12: track 0.00 -> 55.4 mm
- net /595SCLK: track 0.00 -> 51.2 mm
- net /nano_D13: track 0.00 -> 48.3 mm
- net /595RCLK: track 0.00 -> 46.4 mm
- net /nano_D9: track 0.00 -> 46.0 mm
- net /nano_D6: track 0.00 -> 34.7 mm
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Other:
- board size 108.2 x 63.1 mm -> 105 x 64.9 mm
- board text added: "+"
- board text added: "-"
- board text added: "A0"
- board text added: "A1"
- board text added: "A2"
- board text added: "A3"
- board text added: "A6"
- board text added: "A7"
- board text added: "D12"
- board text added: "D13"
- board text added: "D2"
- board text added: "D5"
- board text added: "D6"
- board text added: "D9"
- board text added: "ESP32cam"
- board text added: "G"
- board text added: "J13"
- board text added: "LB"
- board text added: "LF"
- board text added: "Power (12V)"
- board text added: "RB"
- board text added: "RF"
- board text added: "S"
- board text added: "V"
- board text added: "boot"
- board text added: "designed by kw404"
- board text added: "fdtd_studio"
- board text added: "m5"
- board text added: "m6"
- board text added: "motor5_speed"
- board text added: "motor6_speed"
- board text added: "wheel_speed"

Commit message: update
Parts:
- moved J20 6.10 mm to (131.4, 57.8)
Routing:
- net GND: track 363.0 -> 403.7 mm
- net /motor6_speed: track 122.5 -> 98.9 mm
- net +12V: track 118.4 -> 127.7 mm
- net /tilt-: track 14.3 -> 7.81 mm
- net /tilt+: track 13.3 -> 7.25 mm
- net /motor5_speed: track 84.3 -> 85.8 mm
- net +5V: track 268.2 -> 269.3 mm
- net /SCL: track 58.5 -> 59.2 mm
- net /motor3_A: track 27.2 -> 27.9 mm
- net /motorLF-: track 30.0 -> 30.6 mm
- net /wheel_speed: track 147.2 -> 146.6 mm
Other:
- board size 105 x 64.9 mm -> 99.9 x 64.9 mm
