File: circuit/機電整合.kicad_sch (KiCad schematic)
At the start: 38 parts, among them J1 Screw_Terminal_01x02, J10 Conn_01x03, J11 Conn_01x03, J12 Conn_01x03, J13 Conn_01x03, J14 Conn_01x06, J15 Screw_Terminal_01x02, J16 Screw_Terminal_01x02, J17 Screw_Terminal_01x02, J18 Screw_Terminal_01x02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

Commit message: k
Parts:
- U3, U4, U5, U6, U7: footprint Package_DIP:DIP-16_W7.62mm -> Package_DIP:DIP-16_W7.62mm_Socket
Changed lines of the file:
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@@
       (effects (font (size 1.27 1.27)) (justify left))
     )
-    (property "Footprint" "Package_DIP:DIP-16_W7.62mm" (at 152.4 53.34 0)
+    (property "Footprint" "Package_DIP:DIP-16_W7.62mm_Socket" (at 152.4 53.34 0)
       (effects (font (size 1.27 1.27)) hide)
     )
@@
       (effects (font (size 1.27 1.27)) (justify left))
     )
-    (property "Footprint" "Package_DIP:DIP-16_W7.62mm" (at 205.74 139.7 0)
+    (property "Footprint" "Package_DIP:DIP-16_W7.62mm_Socket" (at 205.74 139.7 0)
       (effects (font (size 1.27 1.27)) (justify left) hide)
     )
@@
       (effects (font (size 1.27 1.27)) (justify left))
     )
-    (property "Footprint" "Package_DIP:DIP-16_W7.62mm" (at 105.41 53.34 0)
+    (property "Footprint" "Package_DIP:DIP-16_W7.62mm_Socket" (at 105.41 53.34 0)
       (effects (font (size 1.27 1.27)) hide)
     )
@@
       (effects (font (size 1.27 1.27)) (justify left))
     )
-    (property "Footprint" "Package_DIP:DIP-16_W7.62mm" (at 265.43 139.7 0)
+    (property "Footprint" "Package_DIP:DIP-16_W7.62mm_Socket" (at 265.43 139.7 0)
       (effects (font (size 1.27 1.27)) (justify left) hide)
     )
@@
       (effects (font (size 1.27 1.27)) (justify left))
     )
-    (property "Footprint" "Package_DIP:DIP-16_W7.62mm" (at 208.28 71.12 0)
+    (property "Footprint" "Package_DIP:DIP-16_W7.62mm_Socket" (at 208.28 71.12 0)
       (effects (font (size 1.27 1.27)) (justify left) hide)
     )
