File: circuit/機電整合.kicad_sch (KiCad schematic)
At the start: 7 parts, among them U1 L293D, U2 74HC595, U3 74HC595, U4 L293D, U5 L293D, U6 ESP32-CAM

Commit message: update circuit diagram
Parts:
- added D1, D2, D3: LED, LED_THT:LED_D3.0mm_FlatTop, symbol Device:LED
- added J2: Conn_01x08, Connector_PinHeader_2.54mm:PinHeader_1x08_P2.54mm_Vertical, symbol Connector_Generic:Conn_01x08
- added R1, R2, R3: 200, LED_THT:LED_D3.0mm_FlatTop, symbol Device:R
- added R4: 1k, symbol Device:R
Connections:
- net GND: now also U6.12 (GND_2), U6.7 (GND_1), J2.1 (Pin_1), J2.3 (Pin_3), R1.2, R2.2, R3.2
- net motor5_speed: now also D2.2 (A)
- net motor6_speed: now also D3.2 (A)
- net wheel_speed: now also D1.2 (A)
- net at A1.1 (D1/TX): now also R4.2
- net nano_RX: now reaches A1.2 (D0/RX)
- net nano_RX: now also J2.7 (Pin_7)
- net nano_reset: now reaches A1.3 (~{RESET})
- net nano_reset: now also J2.4 (Pin_4)
- net esp32_GPI0: now reaches U6.11 (IO0)
- net esp32_GPI0: now also J2.2 (Pin_2)
- net esp32_RX: now reaches U6.14 (U0R)
- net esp32_RX: now also J2.6 (Pin_6)
- net esp32_TX: now reaches U6.15 (U0T)
- net esp32_TX: now also J2.8 (Pin_8)
- net motorLb- renamed motorLB-
- new net: D3.1 (K), R3.1
- new net: D2.1 (K), R2.1
- new net: D1.1 (K), R1.1
- new net nano_TX: J2.5 (Pin_5), R4.1
Other:
- moved on the sheet: A1, U1, U2, U3, U4, U5, U6

Commit message: nano pinout
Parts:
- added J10, J11, J12, J13, J14, J15, J16, J17, J18, J19, J8, J9: Conn_01x03, Connector_PinHeader_2.54mm:PinHeader_1x03_P2.54mm_Vertical, symbol Connector_Generic:Conn_01x03
- added J2, J3, J4, J5, J6, J7: Screw_Terminal_01x02, symbol Connector:Screw_Terminal_01x02
- renumbered J2 to J1
Connections:
- net +12V: no longer U1.8 (VCC2), U4.8 (VCC2), U5.8 (VCC2)
- net +5V: now also U1.8 (VCC2), U4.8 (VCC2), U5.8 (VCC2), J10.2 (Pin_2), J11.2 (Pin_2), J12.2 (Pin_2), J13.2 (Pin_2), J14.2 (Pin_2), J15.2 (Pin_2), J16.2 (Pin_2), J17.2 (Pin_2), J18.2 (Pin_2), J19.2 (Pin_2), J8.2 (Pin_2), J9.2 (Pin_2)
- net GND: now also J10.3 (Pin_3), J11.3 (Pin_3), J12.3 (Pin_3), J13.3 (Pin_3), J14.3 (Pin_3), J15.3 (Pin_3), J16.3 (Pin_3), J17.3 (Pin_3), J18.3 (Pin_3), J19.3 (Pin_3), J8.3 (Pin_3), J9.3 (Pin_3)
- net motorLB+: now also J4.1 (Pin_1)
- net motorLB-: now also J4.2 (Pin_2)
- net motorLF+: now also J2.1 (Pin_1)
- net motorLF-: now also J2.2 (Pin_2)
- net motorRB+: now also J5.1 (Pin_1)
- net motorRB-: now also J5.2 (Pin_2)
- net motorRF+: now also J3.1 (Pin_1)
- net motorRF-: now also J3.2 (Pin_2)
- net shoot+: now also J6.1 (Pin_1)
- net shoot-: now also J6.2 (Pin_2)
- net tilt+: now also J7.1 (Pin_1)
- net tilt-: now also J7.2 (Pin_2)
- net nano_D9: now reaches A1.12 (D9)
- net nano_D9: now also J11.1 (Pin_1)
- net nano_D12: now reaches A1.15 (D12)
- net nano_D12: now also J12.1 (Pin_1)
- net nano_D13: now reaches A1.16 (D13)
- net nano_D13: now also J13.1 (Pin_1)
- net nano_A0: now reaches A1.19 (A0)
- net nano_A0: now also J14.1 (Pin_1)
- net nano_A1: now reaches A1.20 (A1)
- net nano_A1: now also J15.1 (Pin_1)
- net nano_A2: now reaches A1.21 (A2)
- net nano_A2: now also J16.1 (Pin_1)
- net nano_A3: now reaches A1.22 (A3)
- net nano_A3: now also J17.1 (Pin_1)
- net nano_A6: now reaches A1.25 (A6)
- net nano_A6: now also J18.1 (Pin_1)
- net nano_A7: now reaches A1.26 (A7)
- net nano_A7: now also J19.1 (Pin_1)
- net nano_D2: now reaches A1.5 (D2)
- net nano_D2: now also J8.1 (Pin_1)
- net nano_D5: now reaches A1.8 (D5)
- net nano_D5: now also J9.1 (Pin_1)
- net nano_D6: now reaches A1.9 (D6)
- net nano_D6: now also J10.1 (Pin_1)
Other:
- moved on the sheet: U4, U5

Commit message: update
Parts:
- removed J14, J15, J16, J17, J18, J19: Conn_01x03, Connector_PinHeader_2.54mm:PinHeader_1x03_P2.54mm_Vertical, symbol Connector_Generic:Conn_01x03
- added C1, C2, C3: C, Capacitor_THT:C_Disc_D5.0mm_W2.5mm_P5.00mm, symbol Device:C
- added J14: Conn_01x06, Connector_PinHeader_2.54mm:PinHeader_1x06_P2.54mm_Vertical, symbol Connector_Generic:Conn_01x06
- added J15: Screw_Terminal_01x02, Connector:HANDSON_KF301-2P, symbol Connector:Screw_Terminal_01x02
- added J16, J17: Conn_01x08, Connector_PinHeader_2.54mm:PinHeader_1x08_P2.54mm_Vertical, symbol Connector_Generic:Conn_01x08
- added U7: LM7805_TO220, Package_TO_SOT_THT:TO-220-3_Vertical, symbol Regulator_Linear:LM7805_TO220
- J2, J3, J4, J5, J6, J7: footprint (none) -> Connector:HANDSON_KF301-2P
- R1, R2, R3: footprint LED_THT:LED_D3.0mm_FlatTop -> Resistor_THT:R_Axial_DIN0207_L6.3mm_D2.5mm_P7.62mm_Horizontal
- R4: footprint (none) -> Resistor_THT:R_Axial_DIN0309_L9.0mm_D3.2mm_P12.70mm_Horizontal
- U6: footprint ESP32-CAM -> Module:ESP32-CAM
Connections:
- net +12V: now also C1.2, C2.2, C3.2, J15.1 (Pin_1), U7.1 (VI); no longer A1.30 (VIN)
- net +5V: now also J16.1 (Pin_1), U7.3 (VO); no longer U6.8 (5V)
- net GND: now also C1.1, C2.1, C3.1, J15.2 (Pin_2), J16.2 (Pin_2), J17.1 (Pin_1), J17.5 (Pin_5), U7.2 (GND); no longer U6.12 (GND_2), U6.16 (GND_3), U6.7 (GND_1)
- net SCL: now also J16.4 (Pin_4); no longer U6.5 (IO13)
- net SDA: now also J16.5 (Pin_5); no longer U6.4 (IO15)
- net esp32_GPI0: now also J17.6 (Pin_6); no longer U6.11 (IO0)
- net esp32_RX: now also J17.3 (Pin_3); no longer U6.14 (U0R)
- net esp32_TX: now also J17.2 (Pin_2); no longer U6.15 (U0T)
- net nano_A0: now also J14.1 (Pin_1)
- net nano_A1: now also J14.2 (Pin_2)
- net nano_A2: now also J14.3 (Pin_3)
- net nano_A3: now also J14.4 (Pin_4)
- net nano_A6: now also J14.5 (Pin_5)
- net nano_A7: now also J14.6 (Pin_6)
- net +3.3V: no longer names the net of U6.9 (3V3)
- net +3.3V: no longer A1.17 (3V3)
- no-connect marks 0 -> 32
Other:
- moved on the sheet: J1

Commit message: pcb done
Parts:
- removed J1: Conn_01x08, Connector_PinHeader_2.54mm:PinHeader_1x08_P2.54mm_Vertical, symbol Connector_Generic:Conn_01x08
- added J4, J5, J6, J7: Conn_01x02, Connector_PinHeader_2.54mm:PinHeader_1x02_P2.54mm_Vertical, symbol Connector_Generic:Conn_01x02
- C1: value C -> 10uf; footprint Capacitor_THT:C_Disc_D5.0mm_W2.5mm_P5.00mm -> Capacitor_THT:CP_Radial_D5.0mm_P2.50mm; symbol Device:C -> Device:C_Polarized_US
- C2: renamed from C3; value C -> 10uf; footprint Capacitor_THT:C_Disc_D5.0mm_W2.5mm_P5.00mm -> Capacitor_THT:CP_Radial_D5.0mm_P2.50mm; symbol Device:C -> Device:C_Polarized_US
- C3: renamed from C2; value C -> 10uf; footprint Capacitor_THT:C_Disc_D5.0mm_W2.5mm_P5.00mm -> Capacitor_THT:CP_Radial_D5.0mm_P2.50mm; symbol Device:C -> Device:C_Polarized_US
- R1: renamed from R4; footprint Resistor_THT:R_Axial_DIN0309_L9.0mm_D3.2mm_P12.70mm_Horizontal -> Resistor_THT:R_Axial_DIN0207_L6.3mm_D2.5mm_P10.16mm_Horizontal
- R2: renamed from R1; value 200 -> 220; footprint Resistor_THT:R_Axial_DIN0207_L6.3mm_D2.5mm_P7.62mm_Horizontal -> Resistor_THT:R_Axial_DIN0207_L6.3mm_D2.5mm_P10.16mm_Horizontal
- R3: renamed from R2; value 200 -> 220; footprint Resistor_THT:R_Axial_DIN0207_L6.3mm_D2.5mm_P7.62mm_Horizontal -> Resistor_THT:R_Axial_DIN0207_L6.3mm_D2.5mm_P10.16mm_Horizontal
- R4: renamed from R3; value 200 -> 220; footprint Resistor_THT:R_Axial_DIN0207_L6.3mm_D2.5mm_P7.62mm_Horizontal -> Resistor_THT:R_Axial_DIN0207_L6.3mm_D2.5mm_P10.16mm_Horizontal
- renumbered J15 to J1, J2 to J15, J3 to J16, J4 to J17, J5 to J18, J6 to J19, J16 to J2, J7 to J20, J17 to J3, U6 to U1, U7 to U2, U2 to U3, U3 to U4, U4 to U5, U1 to U6, U5 to U7
Connections:
- net +12V: now also C1.1, C2.1, C3.1; no longer C1.2, C2.2, C3.2
- net GND: now also C1.2, C2.2, C3.2, J6.1 (Pin_1), J7.1 (Pin_1); no longer C1.1, C2.1, C3.1
- net esp32_GPI0: now also J7.2 (Pin_2)
- net esp32_RX: now also J5.2 (Pin_2)
- net esp32_TX: now also J4.2 (Pin_2)
- net nano_RX: now also J4.1 (Pin_1)
- net nano_TX: now also J5.1 (Pin_1)
- net nano_reset: now also J6.2 (Pin_2)
Other:
- moved on the sheet: U1
